File: Secondary Board/Secondary Board.kicad_sch (KiCad schematic)
At the start: 8 parts, among them J1 USB4145-03-0070-C, J3 5023520500

Commit message: Initial Commit
Parts:
- removed J3: 5023520500, 5023520500:CONN05_502352_MOL, symbol 5023520500:5023520500
- removed S2: TL1014BF220QG, TL10:TL1014BF220QG, symbol TL1014BF220QG:TL1014BF220QG
- added J2: 5023520500, 5023520500:CONN05_502352_MOL, symbol 5023520500:5023520500
- added S1: TL1014BF220QG, TL10:TL1014BF220QG, symbol TL1014BF220QG:TL1014BF220QG
Connections:
- net GND: now also J2.4, S1.2, S1.4
- net SIG: now also J2.1, S1.1, S1.3
- net USB_N: now also J2.2
- net USB_P: now also J2.3
- net VBUS: now also J2.5
